File: hardware/src/dpx_pd_pooper/dpx_pd_pooper.kicad_pcb (KiCad board)
At the start: 2 copper layers, 35 x 25 mm, 19 parts, among them J2 VOUT, SW1 SW_DIP_x03

Commit message: updated production files
qr code and some fixes
Parts:
- removed U1: ~, Package_SO:SSOP-10-1EP_3.9x4.9mm_P1mm_EP2.1x3.3mm_ThermalVias
- turned R6 to 90 degrees
Routing:
- net VDD: track 36.7 -> 36.2 mm

Commit message: lol missing the CH224K ?
Parts:
- removed the SYM1 at (68.1, 73.4)
- added U1: CH224K, Package_SO:SSOP-10-1EP_3.9x4.9mm_P1mm_EP2.1x3.3mm_ThermalVias, F.Cu at (54.6, 65.3)
